Commit message: Fix gripper direction/range and RViz visualization
- Gripper: use grip_level with inverted ESP32 mapping for correct
  direction match between RViz (+120°) and real robot (0-120°)
- URDF gripper axis -1 with limits [-2.0944, 0] for positive RViz rotation
- Add GRIPPER_ESP32_SCALE=1.5 mapping grip level to ESP32 servo range
- teleop publishes odom TF (dead reckoning) to avoid conflict with relay
- RViz fixed frame set to odom, arm/gripper publishers active in both modes
- Increase default turn_speed to 2.0 for ESP32 motor dead zone

File: urdf/rasp_roarm.xacro (robot description, xacro)
@@ -341,6 +341,6 @@
     <parent link="arm_link3" />
     <child link="arm_gripper_link" />
-    <axis xyz="0 0 1" />
-    <limit lower="0" upper="1.5" effort="2" velocity="1.0" />
+    <axis xyz="0 0 -1" />
+    <limit lower="-2.0944" upper="0" effort="2" velocity="1.0" />
     <dynamics damping="1.5" friction="0.3"/>
   </joint>

File: urdf/ugv_roarm.xacro (robot description, xacro)
@@ -371,6 +371,6 @@
     <parent link="arm_link3" />
     <child link="arm_gripper_link" />
-    <axis xyz="0 0 1" />
-    <limit lower="0" upper="1.5" effort="2" velocity="1.0" />
+    <axis xyz="0 0 -1" />
+    <limit lower="-2.0944" upper="0" effort="2" velocity="1.0" />
     <dynamics damping="1.5" friction="0.3"/>
   </joint>
